Commit message: pid

File: ajgar_description/urdf/arm.urdf (robot description, URDF)
Before this commit: robot ajgar, 7 links, 6 joints
Links:
- added link Station_v3_v1_1, mass 84.44124651406766; collision mesh filename=package://ajgar_description/meshes/Station_v3_v1_1.stl scale=0.001 0.001 0.001; visual mesh filename=package://ajgar_description/meshes/Station_v3_v1_1.stl scale=0.001 0.001 0.001
- added link table_v1_1, mass 353.24999999999994; collision mesh filename=package://ajgar_description/meshes/table_v1_1.stl scale=0.001 0.001 0.001; visual mesh filename=package://ajgar_description/meshes/table_v1_1.stl scale=0.001 0.001 0.001
- link base_link: mass None -> 9.059758934586307
- link base_top_1: mass None -> 1.4850383611977547
- link elbow_1: mass None -> 2.4072821039747727
- link end__1: mass None -> 0.07630173554088619
- link shoulder_1: mass None -> 2.8383656665985857
- link suction_1: mass None -> 0.6053245769138885
- link wrist_1: mass None -> 0.34678950211541076
Joints:
- removed joint arm_joint 
- added joint Rigid 8: type fixed, parent base_link, child table_v1_1, origin xyz=-0.015013 0.0 0.0 rpy=0 0 0
- added joint Rigid 9: type fixed, parent table_v1_1, child Station_v3_v1_1, origin xyz=0.0 0.0 -0.025 rpy=0 0 0
- added joint arm_joint: type continuous, parent shoulder_1, child elbow_1, origin xyz=-0.111716 -0.064499 0.223432 rpy=0 0 0, axis 0.5 -0.866025 -0.0
- joint forearm_joint: limit lower=-3.1416 upper=3.1416 effort=5 velocity=1.0 -> (none); type revolute -> continuous
- joint shoulder_joint: limit lower=-1.916 upper=0.606 effort=5 velocity=1.0 -> (none); type revolute -> continuous

File: ajgar_description/urdf/ik_arm.urdf (robot description, URDF)
Before this commit: robot ajgar, 9 links, 8 joints
Links:
- removed link Station_v3_v1_1
- removed link table_v1_1
- link base_link: mass 9.059758934586307 -> None; geometry collision mesh filename=package://ajgar_description/meshes/base_link.stl scale=0.001 0.001 0.001; visual mesh filename=package://ajgar_description/meshes/base_link.stl scale=0.001 0.001 0.001
- link base_top_1: mass 1.4850383611977547 -> None; geometry collision mesh filename=package://ajgar_description/meshes/base_top_1.stl scale=0.001 0.001 0.001; visual mesh filename=package://ajgar_description/meshes/base_top_1.stl scale=0.001 0.001 0.001
- link elbow_1: mass 2.4072821039747727 -> None; geometry collision mesh filename=package://ajgar_description/meshes/elbow_1.stl scale=0.001 0.001 0.001; visual mesh filename=package://ajgar_description/meshes/elbow_1.stl scale=0.001 0.001 0.001
- link end__1: mass 0.07630173554088619 -> None; geometry collision mesh filename=package://ajgar_description/meshes/end__1.stl scale=0.001 0.001 0.001; visual mesh filename=package://ajgar_description/meshes/end__1.stl scale=0.001 0.001 0.001
- link shoulder_1: mass 2.8383656665985857 -> None; geometry collision mesh filename=package://ajgar_description/meshes/shoulder_1.stl scale=0.001 0.001 0.001; visual mesh filename=package://ajgar_description/meshes/shoulder_1.stl scale=0.001 0.001 0.001
- link suction_1: mass 0.6053245769138885 -> None; geometry collision mesh filename=package://ajgar_description/meshes/suction_1.stl scale=0.001 0.001 0.001; visual mesh filename=package://ajgar_description/meshes/suction_1.stl scale=0.001 0.001 0.001
- link wrist_1: mass 0.34678950211541076 -> None; geometry collision mesh filename=package://ajgar_description/meshes/wrist_1.stl scale=0.001 0.001 0.001; visual mesh filename=package://ajgar_description/meshes/wrist_1.stl scale=0.001 0.001 0.001
Joints:
- removed joint Rigid 8
- removed joint Rigid 9
- joint arm_joint: limit (none) -> lower=-1000 upper=1000 effort=5 velocity=1.0; type continuous -> revolute
- joint forearm_joint: limit (none) -> lower=-1000 upper=1000 effort=5 velocity=1.0; type continuous -> revolute
- joint shoulder_joint: limit (none) -> lower=-1000 upper=1000 effort=5 velocity=1.0; type continuous -> revolute
